File: Clone/Board/Eagle/Jupiter Ace build024.brd (EAGLE design)
At the start: 209 x 184 mm, 325 parts, among them K1 1, K10 0, K11 Q, K12 W, K13 E, K14 R, K15 T, K16 Y, K17 U, K18 I, K19 O, K2 2, K20 P, K21 A, K22 S, K23 D, K24 F, K25 G, K26 H, K27 J, K28 K, K29 L, K3 3, K30 ENTER, K31 SHIFT, K32 SYMBOL, K33 Z, K34 X, K35 C, K36 V, K37 B, K38 N, K39 M, K4 4, K40 SPACE, K41 SPACE, K5 5, K6 6, K7 7, K8 8, K9 9, Q1 2N3904, Q3 BC337, U1 7805, U2 MAX4390EUK, X1 6.5MHz, X2 CON-CONRAD_736880-49

Commit message: BUILD 024
Parts:
- JP9: value KEYBOARD -> ACE81 SELECTOR
- R42: value 10K -> 1KB
Connections:
- removed net N$126: JP9.2, Z40.1
- net ACE81_ENABLED: now also JP9.2, Z40.1; no longer JP9.3
- net GND: now also JP9.3
Routing:
- net ACE81_ENABLED: track 349.9 -> 404.1 mm
- net N$126: track 51.8 -> 0.00 mm
- net GND: track 1385.0 -> 1389.0 mm
Other:
- board text added: "2022 Alejandro Valero Sebastián & Pedro Gimeno Fortea Mercury Ace v1.0 (Build 24)"
- board text added: "ACE81 ON"
- board text removed: "2022 Alejandro Valero Sebastián & Pedro Gimeno Fortea Mercury Ace v1.0 (Build 23)"
- board text removed: "KBD 81"
Changed lines of the file:
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@@
 </layers>
 <board>
-<fusionsync huburn="a.YnVzaW5lc3M6aG90bWFpbDM5ODA5NQ" projecturn="a.YnVzaW5lc3M6aG90bWFpbDM5ODA5NSNEMjAyMzA0MDQ2Mjc4MjA0MjY" f3durn="urn:adsk.wipprod:dm.lineage:SZGlU60bTwWuY3Eq3Hediw" pcbguid="" lastpulledtime="" lastsyncedchangeguid="" latestrevisionid="78e4683f-c3d4-49d7-9e59-0e025e3c7355" lastsyncedrevisionid="78e4683f-c3d4-49d7-9e59-0e025e3c7355" lastboardhashguid="bc6eac52-4dc6-b687-9bc6-3bf55017709d" lastpushedtime="2023-08-20T14:22:14Z" linktopcb3d="true"/>
+<fusionsync huburn="a.YnVzaW5lc3M6aG90bWFpbDM5ODA5NQ" projecturn="a.YnVzaW5lc3M6aG90bWFpbDM5ODA5NSNEMjAyMzA0MDQ2Mjc4MjA0MjY" f3durn="urn:adsk.wipprod:dm.lineage:SZGlU60bTwWuY3Eq3Hediw" pcbguid="" lastpulledtime="" lastsyncedchangeguid="" latestrevisionid="78e4683f-c3d4-49d7-9e59-0e025e3c7355" lastsyncedrevisionid="78e4683f-c3d4-49d7-9e59-0e025e3c7355" lastboardhashguid="bc6eac52-4dc6-b687-9bc6-3bf55017709d" lastpushedtime="2023-08-20T14:22:14Z" linktopcb3d="false"/>
 <plain>
 <wire x1="0" y1="5.388153125" x2="0" y2="182.306690625" width="0" layer="20"/>
@@
 <wire x1="209" y1="88" x2="0" y2="88" width="0" layer="41"/>
 <wire x1="209" y1="88" x2="0" y2="88" width="0" layer="42"/>
-<text x="25.4" y="1.27" size="1.905" layer="25">   2022 Alejandro Valero Sebastián &amp; Pedro Gimeno Fortea Mercury Ace v1.0 (Build 23)</text>
+<text x="25.4" y="1.27" size="1.905" layer="25">   2022 Alejandro Valero Sebastián &amp; Pedro Gimeno Fortea Mercury Ace v1.0 (Build 24)</text>
 <text x="107.95" y="171.45" size="1.016" layer="25">R16..R20</text>
 <text x="134.62" y="166.37" size="1.016" layer="25">R12..R15</text>
@@
 <text x="0" y="-0.127" size="0.0508" layer="201" font="vector">C:/Users/aleja/OneDrive/Documentos/Mercury Ace_.bmp</text>
 <text x="0.508" y="92.202" size="0.8128" layer="27" rot="R270" align="center-right">KBD AUTO</text>
-<text x="0.635" y="85.09" size="1.016" layer="27" rot="R270" align="center-right">KBD 81</text>
+<text x="0.635" y="85.09" size="1.016" layer="27" rot="R270" align="center-right">ACE81 ON</text>
 <text x="201.041" y="91.186" size="1.778" layer="21">+</text>
 <text x="9.398" y="92.202" size="1.778" layer="21">+</text>
@@
 <attribute name="NAME" x="196.723" y="169.672" size="1.27" layer="25" rot="R180"/>
 </element>
-<element name="JP9" library="pinhead" library_urn="urn:adsk.eagle:library:325" package="1X03" package3d_urn="urn:adsk.eagle:package:22458/2" value="KEYBOARD" x="2.54" y="92.202" smashed="yes" rot="R90">
+<element name="JP9" library="pinhead" library_urn="urn:adsk.eagle:library:325" package="1X03" package3d_urn="urn:adsk.eagle:package:22458/2" value="ACE81 SELECTOR" x="2.54" y="92.202" smashed="yes" rot="R90">
 <attribute name="NAME" x="4.445" y="96.774" size="1.27" layer="25" ratio="10" rot="R270"/>
 <attribute name="POPULARITY" value="92" x="2.54" y="92.202" size="1.778" layer="27" rot="R90" display="off"/>
@@
 <element name="U$41" library="switch-omron" library_urn="urn:adsk.eagle:library:40469038" package="CARBONB3F" package3d_urn="urn:adsk.eagle:package:41369143/6" value="40-XX-CARBON" x="194.564" y="17" smashed="yes" rot="R90"/>
 <element name="U$42" library="switch-omron" library_urn="urn:adsk.eagle:library:40469038" package="CARBONB3F" package3d_urn="urn:adsk.eagle:package:41369143/6" value="40-XX-CARBON" x="200.3" y="17" smashed="yes" rot="R270"/>
-<element name="R42" library="rcl" library_urn="urn:adsk.eagle:library:334" package="0204/7" package3d_urn="urn:adsk.eagle:package:23498/2" value="10K" x="138.1125" y="154.94" smashed="yes" rot="R180">
+<element name="R42" library="rcl" library_urn="urn:adsk.eagle:library:334" package="0204/7" package3d_urn="urn:adsk.eagle:package:23498/2" value="1KB" x="138.1125" y="154.94" smashed="yes" rot="R180">
 <attribute name="NAME" x="140.6525" y="153.6446" size="0.9906" layer="25" ratio="10" rot="R180"/>
 <attribute name="POPULARITY" value="79" x="138.1125" y="154.94" size="1.778" layer="27" rot="R180" display="off"/>
@@
 <wire x1="12.3656" y1="104.4956" x2="7.62" y2="99.75" width="0.4064" layer="1"/>
 <wire x1="21.1994" y1="104.4956" x2="12.3656" y2="104.4956" width="0.4064" layer="1"/>
+<contactref element="JP9" pad="3"/>
+<wire x1="2.54" y1="94.742" x2="4.953" y2="92.329" width="0.4" layer="16"/>
+<wire x1="4.953" y1="92.329" x2="5.588" y2="92.329" width="0.4" layer="16"/>
 </signal>
 <signal name="VCC" class="1">
@@
 <wire x1="46" y1="123.75" x2="46.25" y2="123.75" width="0.4" layer="1"/>
 <wire x1="4.5" y1="91.5" x2="2.75" y2="89.75" width="0.4" layer="1"/>
+<wire x1="5.77" y1="94.52" x2="4.5" y2="93.25" width="0.4" layer="1"/>
 <wire x1="4.5" y1="93.25" x2="4.5" y2="91.5" width="0.4" layer="1"/>
-<wire x1="7.75" y1="96.5" x2="4.5" y2="93.25" width="0.4" layer="16"/>
+<wire x1="7.75" y1="96.5" x2="5.77" y2="94.52" width="0.4" layer="16"/>
 <wire x1="2.75" y1="89.75" x2="2.54" y2="89.662" width="0.4" layer="1"/>
 <wire x1="7.75" y1="96.5" x2="7.493" y2="97.155" width="0.4" layer="16"/>
@@
 <via x="59.75" y="131" extent="1-16" drill="0.254"/>
 <via x="46.75" y="115.5" extent="1-16" drill="0.254"/>
-<via x="4.5" y="93.25" extent="1-16" drill="0.254"/>
+<via x="5.77" y="94.52" extent="1-16" drill="0.254"/>
 <via x="90.5" y="177.5" extent="1-16" drill="0.254"/>
 <via x="85.25" y="106.75" extent="1-16" drill="0.254"/>
@@
 <contactref element="Z1-2" pad="1"/>
 <contactref element="R29" pad="2"/>
-<contactref element="JP9" pad="3"/>
 <wire x1="166.5" y1="90.25" x2="177.5" y2="90.25" width="0.254" layer="16"/>
 <wire x1="156.5" y1="90.25" x2="166.5" y2="90.25" width="0.254" layer="1"/>
@@
 <wire x1="12.5" y1="120.75" x2="14.75" y2="123" width="0.254" layer="1"/>
 <wire x1="12.5" y1="109.75" x2="12.5" y2="120.75" width="0.254" layer="1"/>
-<wire x1="4.5" y1="101.75" x2="12.5" y2="109.75" width="0.254" layer="1"/>
-<wire x1="4.5" y1="96.5" x2="4.5" y2="101.75" width="0.254" layer="1"/>
-<wire x1="2.75" y1="94.75" x2="4.5" y2="96.5" width="0.254" layer="1"/>
+<wire x1="12.5" y1="109.75" x2="4.5" y2="101.75" width="0.254" layer="1"/>
 <wire x1="35.75" y1="170" x2="35.56" y2="170.18" width="0.254" layer="16"/>
-<wire x1="2.75" y1="94.75" x2="2.54" y2="94.742" width="0.254" layer="1"/>
 <wire x1="145" y1="166.5" x2="145" y2="156" width="0.254" layer="16"/>
 <wire x1="86.25" y1="166.5" x2="145" y2="166.5" width="0.254" layer="16"/>
@@
 <wire x1="145" y1="156" x2="135.5" y2="156" width="0.1524" layer="16"/>
 <wire x1="134.5" y1="155" x2="134.3025" y2="154.94" width="0.1524" layer="16"/>
+<contactref element="Z40" pad="1"/>
+<contactref element="JP9" pad="2"/>
+<wire x1="14.192" y1="48.768" x2="2.4227" y2="60.5373" width="0.4" layer="16"/>
+<wire x1="2.4227" y1="79.69408125" x2="2.4227" y2="60.5373" width="0.4" layer="16"/>
+<wire x1="2.4227" y1="79.69408125" x2="6.731" y2="84.00238125" width="0.4" layer="16"/>
+<wire x1="6.731" y1="84.00238125" x2="6.731" y2="88.011" width="0.4" layer="16"/>
+<wire x1="6.731" y1="88.011" x2="2.54" y2="92.202" width="0.4" layer="16"/>
+<wire x1="4.5" y1="94.162" x2="2.54" y2="92.202" width="0.254" layer="1"/>
+<wire x1="4.5" y1="101.75" x2="4.5" y2="94.162" width="0.254" layer="1"/>
 </signal>
 <signal name="N$32">
@@
 <wire x1="15.5" y1="111.75" x2="15.7" y2="111.96" width="0.254" layer="16"/>
 </signal>
-<signal name="N$126">
-<contactref element="Z40" pad="1"/>
-<contactref element="JP9" pad="2"/>
-<wire x1="14.192" y1="48.768" x2="2.4227" y2="60.5373" width="0.4" layer="16"/>
-<wire x1="2.4227" y1="79.69408125" x2="2.4227" y2="60.5373" width="0.4" layer="16"/>
-<wire x1="2.4227" y1="79.69408125" x2="6.731" y2="84.00238125" width="0.4" layer="16"/>
-<wire x1="6.731" y1="84.00238125" x2="6.731" y2="88.011" width="0.4" layer="16"/>
-<wire x1="6.731" y1="88.011" x2="2.54" y2="92.202" width="0.4" layer="16"/>
-</signal>
 <signal name="N$16">

Commit message: doc build024
Parts:
- R42: value 1KB -> 1K
Routing:
- net ACE81_ENABLED: track 404.1 -> 402.7 mm
Other:
- board text added: "2022 Alejandro Valero Sebastián & Pedro Gimeno Fortea Mercury Ace v1.0 (Build 23)"
- board text added: "R11..R15,R42"
- board text removed: "2022 Alejandro Valero Sebastián & Pedro Gimeno Fortea Mercury Ace v1.0 (Build 24)"
- board text removed: "R12..R15"
Changed lines of the file:
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@@
 </layers>
 <board>
-<fusionsync huburn="a.YnVzaW5lc3M6aG90bWFpbDM5ODA5NQ" projecturn="a.YnVzaW5lc3M6aG90bWFpbDM5ODA5NSNEMjAyMzA0MDQ2Mjc4MjA0MjY" f3durn="urn:adsk.wipprod:dm.lineage:SZGlU60bTwWuY3Eq3Hediw" pcbguid="" lastpulledtime="" lastsyncedchangeguid="" latestrevisionid="78e4683f-c3d4-49d7-9e59-0e025e3c7355" lastsyncedrevisionid="78e4683f-c3d4-49d7-9e59-0e025e3c7355" lastboardhashguid="bc6eac52-4dc6-b687-9bc6-3bf55017709d" lastpushedtime="2023-08-20T14:22:14Z" linktopcb3d="false"/>
+<fusionsync huburn="a.YnVzaW5lc3M6aG90bWFpbDM5ODA5NQ" projecturn="a.YnVzaW5lc3M6aG90bWFpbDM5ODA5NSNEMjAyMzA0MDQ2Mjc4MjA0MjY" f3durn="urn:adsk.wipprod:dm.lineage:SZGlU60bTwWuY3Eq3Hediw" pcbguid="" lastpulledtime="" lastsyncedchangeguid="" latestrevisionid="78e4683f-c3d4-49d7-9e59-0e025e3c7355" lastsyncedrevisionid="78e4683f-c3d4-49d7-9e59-0e025e3c7355" lastboardhashguid="bc6eac52-4dc6-b687-9bc6-3bf55017709d" lastpushedtime="2023-08-20T14:22:14Z" linktopcb3d="true"/>
 <plain>
 <wire x1="0" y1="5.388153125" x2="0" y2="182.306690625" width="0" layer="20"/>
@@
 <wire x1="209" y1="88" x2="0" y2="88" width="0" layer="41"/>
 <wire x1="209" y1="88" x2="0" y2="88" width="0" layer="42"/>
-<text x="25.4" y="1.27" size="1.905" layer="25">   2022 Alejandro Valero Sebastián &amp; Pedro Gimeno Fortea Mercury Ace v1.0 (Build 24)</text>
+<text x="25.4" y="1.27" size="1.905" layer="25">   2022 Alejandro Valero Sebastián &amp; Pedro Gimeno Fortea Mercury Ace v1.0 (Build 23)</text>
 <text x="107.95" y="171.45" size="1.016" layer="25">R16..R20</text>
-<text x="134.62" y="166.37" size="1.016" layer="25">R12..R15</text>
+<text x="134.62" y="166.37" size="1.016" layer="25">R11..R15,R42</text>
 <circle x="25.1079" y="2.286" radius="1.6" width="0.1524" layer="27"/>
 <text x="24.1554" y="1.4097" size="2.54" layer="25">c</text>
@@
 </element>
 <element name="R11" library="rcl" library_urn="urn:adsk.eagle:library:334" package="0204/7" package3d_urn="urn:adsk.eagle:package:23498/2" value="1K" x="138.1125" y="152.4" smashed="yes" rot="R180">
-<attribute name="NAME" x="136.2075" y="153.6954" size="0.9906" layer="25" ratio="10"/>
 <attribute name="POPULARITY" value="79" x="138.1125" y="152.4" size="1.778" layer="27" rot="R180" display="off"/>
 <attribute name="SPICEPREFIX" value="R" x="138.1125" y="152.4" size="1.778" layer="27" rot="R180" display="off"/>
@@
 <element name="U$41" library="switch-omron" library_urn="urn:adsk.eagle:library:40469038" package="CARBONB3F" package3d_urn="urn:adsk.eagle:package:41369143/6" value="40-XX-CARBON" x="194.564" y="17" smashed="yes" rot="R90"/>
 <element name="U$42" library="switch-omron" library_urn="urn:adsk.eagle:library:40469038" package="CARBONB3F" package3d_urn="urn:adsk.eagle:package:41369143/6" value="40-XX-CARBON" x="200.3" y="17" smashed="yes" rot="R270"/>
-<element name="R42" library="rcl" library_urn="urn:adsk.eagle:library:334" package="0204/7" package3d_urn="urn:adsk.eagle:package:23498/2" value="1KB" x="138.1125" y="154.94" smashed="yes" rot="R180">
-<attribute name="NAME" x="140.6525" y="153.6446" size="0.9906" layer="25" ratio="10" rot="R180"/>
+<element name="R42" library="rcl" library_urn="urn:adsk.eagle:library:334" package="0204/7" package3d_urn="urn:adsk.eagle:package:23498/2" value="1K" x="138.1125" y="154.94" smashed="yes" rot="R180">
 <attribute name="POPULARITY" value="79" x="138.1125" y="154.94" size="1.778" layer="27" rot="R180" display="off"/>
 <attribute name="SPICEPREFIX" value="R" x="138.1125" y="154.94" size="1.778" layer="27" rot="R180" display="off"/>
@@
 <wire x1="103.75" y1="154.25" x2="103.75" y2="156.5" width="0.254" layer="1"/>
 <wire x1="104.25" y1="153.75" x2="103.75" y2="154.25" width="0.254" layer="16"/>
-<wire x1="134.5" y1="153.75" x2="104.25" y2="153.75" width="0.254" layer="16"/>
-<wire x1="140.75" y1="147.5" x2="134.5" y2="153.75" width="0.254" layer="1"/>
-<wire x1="140.75" y1="144.75" x2="140.75" y2="147.5" width="0.254" layer="1"/>
+<wire x1="135.135" y1="153.75" x2="104.25" y2="153.75" width="0.254" layer="16"/>
+<wire x1="140.75" y1="148.135" x2="135.135" y2="153.75" width="0.254" layer="1"/>
+<wire x1="140.75" y1="144.75" x2="140.75" y2="148.135" width="0.254" layer="1"/>
 <wire x1="145.75" y1="139.75" x2="140.75" y2="144.75" width="0.254" layer="16"/>
 <wire x1="165.5" y1="139.75" x2="145.75" y2="139.75" width="0.254" layer="16"/>
@@
 <via x="187.639" y="141" extent="1-16" drill="0.254"/>
 <via x="103.75" y="154.25" extent="1-16" drill="0.254"/>
-<via x="134.5" y="153.75" extent="1-16" drill="0.254"/>
+<via x="135.135" y="153.75" extent="1-16" drill="0.254"/>
 <via x="140.75" y="144.75" extent="1-16" drill="0.254"/>
 </signal>
@@
 <wire x1="153.25" y1="156" x2="153.5" y2="155.75" width="0.254" layer="16"/>
 <wire x1="145" y1="156" x2="153.25" y2="156" width="0.254" layer="16"/>
-<wire x1="144" y1="155" x2="145" y2="156" width="0.254" layer="16"/>
 <wire x1="177.5" y1="90.25" x2="177.546" y2="90.17" width="0.254" layer="16"/>
 <wire x1="36.5" y1="169.25" x2="35.75" y2="170" width="0.254" layer="16"/>
