File: Clone/Board/Eagle/Jupiter Ace build024.brd (EAGLE design)
At the start: 209 x 184 mm, 325 parts, among them K1 1, K10 0, K11 Q, K12 W, K13 E, K14 R, K15 T, K16 Y, K17 U, K18 I, K19 O, K2 2, K20 P, K21 A, K22 S, K23 D, K24 F, K25 G, K26 H, K27 J, K28 K, K29 L, K3 3, K30 ENTER, K31 SHIFT, K32 SYMBOL, K33 Z, K34 X, K35 C, K36 V, K37 B, K38 N, K39 M, K4 4, K40 SPACE, K41 SPACE, K5 5, K6 6, K7 7, K8 8, K9 9, Q1 2N3904, Q3 BC337, U1 7805, U2 MAX4390EUK, X1 6.5MHz, X2 CON-CONRAD_736880-49

Commit message: circuit
Parts:
- removed JP9: ACE81 SELECTOR, pinhead:1X03
- added R43: 10K, rcl:0204/7
- S1: value ROMSEL -> (none); device switch-dil:DS-02 -> switch-dil:DP-03
- moved S1 4.02 mm to (59.7, 158.8)
Connections:
- removed net N$33: R34.1, SJ1.1, X2.2, X2.2@2
- net ACE81_ENABLED: now also R43.2, S1.6; no longer JP9.2
- net GND: now also S1.3; no longer JP9.3
- net N$47: now also S1.4; no longer S1.3
- net N$48: now also S1.5; no longer S1.4
- net VCC: now also R43.1; no longer JP9.1
- net VIDEO: now also R34.1, SJ1.1, X2.2, X2.2@2
Routing:
- net VIDEO: track 5.37 -> 79.2 mm, vias 0 -> 1
- net N$33: track 25.0 -> 0.00 mm, vias 1 -> 0
- net A13: track 147.5 -> 171.2 mm, vias 5 -> 9
- net ACE81_ENABLED: track 402.7 -> 419.5 mm, vias 8 -> 10
- net A4: track 164.8 -> 180.1 mm
- net A12: track 170.4 -> 156.1 mm, vias 9 -> 7
- net A3: track 182.0 -> 169.8 mm
- net A11: track 207.4 -> 195.4 mm, vias 6 -> 7
- net A9: track 243.2 -> 253.5 mm, vias 11 -> 12
- net VCC: track 1117.6 -> 1127.4 mm, vias 21 -> 24
- net A6: track 165.8 -> 156.4 mm, vias 8 -> 7
- net D6: track 236.7 -> 229.0 mm, vias 5 -> 4
- net A0: track 211.8 -> 217.9 mm, vias 6 -> 9
- net D2: track 243.1 -> 237.3 mm, vias 12 -> 13
- net N$47: track 7.93 -> 12.8 mm, vias 0 -> 1
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
Commit message: hires-addon
Parts:
- R32, R33: value (none) -> 200
- R34: value (none) -> 75
Changed lines of the file:
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@@
 <attribute name="VALUE" x="199.665" y="18.905" size="0.8128" layer="27" ratio="10" rot="R270"/>
 </element>
-<element name="R32" library="rcl" library_urn="urn:adsk.eagle:library:334" package="0204/7" package3d_urn="urn:adsk.eagle:package:23498/2" value="" x="202.819" y="181.737" smashed="yes" rot="R180">
+<element name="R32" library="rcl" library_urn="urn:adsk.eagle:library:334" package="0204/7" package3d_urn="urn:adsk.eagle:package:23498/2" value="200" x="202.819" y="181.737" smashed="yes" rot="R180">
 <attribute name="NAME" x="202.438" y="180.0606" size="0.9906" layer="25" ratio="10" rot="R180"/>
 <attribute name="POPULARITY" value="79" x="202.819" y="181.737" size="1.778" layer="27" rot="R180" display="off"/>
@@
 <attribute name="VALUE" x="193.38" y="13.825" size="1.27" layer="27" ratio="10" rot="R90"/>
 </element>
-<element name="R33" library="rcl" library_urn="urn:adsk.eagle:library:334" package="0204/7" package3d_urn="urn:adsk.eagle:package:23498/2" value="" x="189.103" y="177.927" smashed="yes" rot="R270">
+<element name="R33" library="rcl" library_urn="urn:adsk.eagle:library:334" package="0204/7" package3d_urn="urn:adsk.eagle:package:23498/2" value="200" x="189.103" y="177.927" smashed="yes" rot="R270">
 <attribute name="NAME" x="187.96" y="171.9834" size="0.9906" layer="25" ratio="10"/>
 <attribute name="POPULARITY" value="79" x="189.103" y="177.927" size="1.778" layer="27" rot="R270" display="off"/>
@@
 <attribute name="VALUE" x="188.6204" y="179.5526" size="0.9906" layer="27" ratio="10" rot="R270"/>
 </element>
-<element name="R34" library="rcl" library_urn="urn:adsk.eagle:library:334" package="0204/7" package3d_urn="urn:adsk.eagle:package:23498/2" value="" x="192.024" y="177.927" smashed="yes" rot="R90">
+<element name="R34" library="rcl" library_urn="urn:adsk.eagle:library:334" package="0204/7" package3d_urn="urn:adsk.eagle:package:23498/2" value="75" x="192.024" y="177.927" smashed="yes" rot="R90">
 <attribute name="NAME" x="193.294" y="172.9486" size="0.9906" layer="25" ratio="10" rot="R180"/>
 <attribute name="POPULARITY" value="79" x="192.024" y="177.927" size="1.778" layer="27" rot="R90" display="off"/>
