File: Clone/Board/Eagle/Jupiter Ace build024.sch (EAGLE design)
At the start: 325 parts, among them K1 1, K10 0, K11 Q, K12 W, K13 E, K14 R, K15 T, K16 Y, K17 U, K18 I, K19 O, K2 2, K20 P, K21 A, K22 S, K23 D, K24 F, K25 G, K26 H, K27 J, K28 K, K29 L, K3 3, K30 ENTER, K31 SHIFT, K32 SYMBOL, K33 Z, K34 X, K35 C, K36 V, K37 B, K38 N, K39 M, K4 4, K40 SPACE, K41 SPACE, K5 5, K6 6, K7 7, K8 8, K9 9, Q1 2N3904, Q3 BC337, U1 7805, U2 MAX4390EUK, X1 6.5MHz, X2 CON-CONRAD_736880-49

Commit message: BUILD 024
Parts:
- JP9: value KEYBOARD -> ACE81 SELECTOR
- R42: value 10K -> 1KB
Connections:
- removed net N$126: JP9.2, Z40.CLK
- net ACE81_ENABLED: now also JP9.2, Z40.CLK; no longer JP9.3
- net GND: now also JP9.3
Other:
- note added: "ACE81 OFF"
- note added: "ACE81 ON"
- note removed: "AUTO"
- note removed: "FORCE81"

Commit message: doc build024
Parts:
- R42: value 1KB -> 1K
Changed lines of the file:
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@@
 <part name="U$41" library="switch-omron" library_urn="urn:adsk.eagle:library:40469038" deviceset="40-XX-CARBON" device="" package3d_urn="urn:adsk.eagle:package:41369143/6"/>
 <part name="U$42" library="switch-omron" library_urn="urn:adsk.eagle:library:40469038" deviceset="40-XX-CARBON" device="" package3d_urn="urn:adsk.eagle:package:41369143/6"/>
-<part name="R42" library="rcl" library_urn="urn:adsk.eagle:library:334" deviceset="R-EU_" device="0204/7" package3d_urn="urn:adsk.eagle:package:23498/2" value="1KB"/>
+<part name="R42" library="rcl" library_urn="urn:adsk.eagle:library:334" deviceset="R-EU_" device="0204/7" package3d_urn="urn:adsk.eagle:package:23498/2" value="1K"/>
 </parts>
 <sheets>
@@
 <wire x1="96.52" y1="-278.13" x2="96.52" y2="-271.78" width="0.1524" layer="91"/>
 <junction x="96.52" y="-271.78"/>
+<junction x="25.4" y="-212.09"/>
 </segment>
 <segment>
@@
 <wire x1="92.964" y1="-208.28" x2="88.9" y2="-208.28" width="0.1524" layer="91"/>
 <junction x="88.9" y="-208.28"/>
+<junction x="40.64" y="-208.28"/>
 </segment>
 <segment>
@@
 <wire x1="288.29" y1="-285.75" x2="288.29" y2="-284.48" width="0.1524" layer="91"/>
 <wire x1="288.29" y1="-284.48" x2="283.21" y2="-284.48" width="0.1524" layer="91"/>
+<junction x="283.21" y="-284.48"/>
 </segment>
 <segment>
@@
 <junction x="152.4" y="-312.42"/>
 <junction x="139.7" y="-312.42"/>
+<label x="124.46" y="-297.18" size="1.778" layer="95"/>
 </segment>
 <segment>

Commit message: circuit
Parts:
- removed JP9: ACE81 SELECTOR, pinhead:PINHD-1X3
- added R43: 10K, rcl:R-EU_0204/7
- S1: value ROMSEL -> (none); device switch-dil:DS02 -> switch-dil:DP03
Connections:
- removed net N$33: R34.1, SJ1.1, X2.1, X2.2@2
- net ACE81_ENABLED: now also R43.2, S1.6; no longer JP9.2
- net GND: now also S1.3; no longer JP9.3
- net N$47: now also S1.4; no longer S1.3
- net N$48: now also S1.5; no longer S1.4
- net VCC: now also R43.1; no longer JP9.1
- net VIDEO: now also R34.1, SJ1.1, X2.1, X2.2@2
Other:
- note removed: "ACE81 OFF"
- note removed: "ACE81 ON"

Commit message: hires-addon
Parts:
- R32, R33: value (none) -> 200
- R34: value (none) -> 75
Changed lines of the file:
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@@
 <part name="GND24" library="supply1" deviceset="GND" device=""/>
 <part name="GND26" library="supply1" deviceset="GND" device=""/>
-<part name="R32" library="rcl" library_urn="urn:adsk.eagle:library:334" deviceset="R-EU_" device="0204/7" package3d_urn="urn:adsk.eagle:package:23498/2"/>
+<part name="R32" library="rcl" library_urn="urn:adsk.eagle:library:334" deviceset="R-EU_" device="0204/7" package3d_urn="urn:adsk.eagle:package:23498/2" value="200"/>
 <part name="K41" library="switch-omron" library_urn="urn:adsk.eagle:library:40469038" deviceset="40-XX" device="NOHOLES" package3d_urn="urn:adsk.eagle:package:40469046/2" value="SPACE"/>
-<part name="R33" library="rcl" library_urn="urn:adsk.eagle:library:334" deviceset="R-EU_" device="0204/7" package3d_urn="urn:adsk.eagle:package:23498/2"/>
-<part name="R34" library="rcl" library_urn="urn:adsk.eagle:library:334" deviceset="R-EU_" device="0204/7" package3d_urn="urn:adsk.eagle:package:23498/2"/>
+<part name="R33" library="rcl" library_urn="urn:adsk.eagle:library:334" deviceset="R-EU_" device="0204/7" package3d_urn="urn:adsk.eagle:package:23498/2" value="200"/>
+<part name="R34" library="rcl" library_urn="urn:adsk.eagle:library:334" deviceset="R-EU_" device="0204/7" package3d_urn="urn:adsk.eagle:package:23498/2" value="75"/>
 <part name="R35" library="rcl" library_urn="urn:adsk.eagle:library:334" deviceset="R-EU_" device="0204/7" package3d_urn="urn:adsk.eagle:package:23498/2" value="300"/>
 <part name="C4" library="rcl" library_urn="urn:adsk.eagle:library:334" deviceset="C-EU" device="025-025X050" package3d_urn="urn:adsk.eagle:package:23629/2" value="100nF"/>
